File: pcb/hypnos/hypnos.kicad_pcb (KiCad board)
At the start: 2 copper layers, 9 parts, among them J1 Shutdown_Switch, J2 User_Input, J3 Debug_Conn, Q1 FDN361BN, SW1 Reset_Switch, U1 RV-3028-C7, U2 BT840F

Commit message: backup work
Parts:
- removed J2: User_Input, Connector_PinHeader_2.54mm:PinHeader_1x02_P2.54mm_Horizontal
- BT1: value BK-883 -> BC-2003-TR; footprint Hypnos:BAT_BK-883 -> Hypnos:BC-2003-TR
- J1: value Shutdown_Switch -> Motherboard_IO; footprint Connector_PinHeader_2.54mm:PinHeader_1x02_P2.54mm_Horizontal -> Hypnos:Conn-Female-RightAnglex3-SMD
- J3: footprint Connector_PinHeader_2.54mm:PinHeader_1x07_P2.54mm_Horizontal -> Hypnos:Conn-Female-RightAnglex7-SMD
- Q1: value FDN361BN -> NDS351NCT; footprint Hypnos:FDN361BN -> Package_TO_SOT_SMD:SOT-323_SC-70_Handsoldering
- moved J3 70.7 mm to (107.2, 122.4), turned to 90 degrees
- moved U2 34.3 mm to (129.4, 110.8), turned to 270 degrees
- moved BT1 32.8 mm to (113.6, 111.0), turned to 270 degrees
- moved U1 30.5 mm to (126.2, 99.9), turned to 90 degrees
- moved C1 22.8 mm to (127.2, 97.0)
- moved Q1 13.4 mm to (120.8, 99.5), turned to 180 degrees
- moved J1 5.90 mm to (101.7, 96.8)
- moved SW1 4.64 mm to (104.3, 101.9), turned to 180 degrees
Connections:
- J1 pad 1: Net-(J1-Pad1) -> /USER_INPUT
- J1 pad 2: Net-(J1-Pad2) -> /OFF_SWITCH
- Q1 pad 1: Net-(Q1-Pad1) -> /OFF_SWITCH_CTRL
- Q1 pad 2: Net-(J1-Pad2) -> GND
- Q1 pad 3: Net-(J1-Pad1) -> /OFF_SWITCH
- U2 pad 11: Net-(U2-Pad11) -> Net-(SW1-Pad1)
- U2 pad 13: Net-(SW1-Pad1) -> Net-(U2-Pad13)
- U2 pad 5: Net-(Q1-Pad1) -> Net-(U1-Pad2)
- U2 pad 6: Net-(J2-Pad1) -> /USER_INPUT
- U2 pad 7: Net-(U1-Pad2) -> /OFF_SWITCH_CTRL
Routing:
- net VDD: track 0.00 -> 64.2 mm, vias 0 -> 4
- net Net-(SW1-Pad1): track 0.00 -> 34.6 mm
- net /SWDIO: track 0.00 -> 27.0 mm
- net /SWDCLK: track 0.00 -> 25.4 mm
- net /~RESET: track 0.00 -> 25.4 mm
- net /USER_INPUT: track 0.00 -> 25.4 mm, vias 0 -> 2
- net GND: track 0.00 -> 23.7 mm, vias 0 -> 8
- net /OFF_SWITCH: track 0.00 -> 17.7 mm
- net Net-(U1-Pad8): track 0.00 -> 8.40 mm, vias 0 -> 2
- net Net-(U1-Pad2): track 0.00 -> 5.87 mm, vias 0 -> 2
- net /OFF_SWITCH_CTRL: track 0.00 -> 4.51 mm
- net Net-(U1-Pad1): track 0.00 -> 4.09 mm
- net Net-(U1-Pad4): track 0.00 -> 3.88 mm
- net Net-(U1-Pad3): track 0.00 -> 3.80 mm
- added copper zone on B.Cu, net GND
Other:
- board outline added: 30 x 30 mm
- net class Default: clearance 0.2 -> 0.26
- rule trace_clearance: 0.2 -> 0.26
- board text added: "Hypnos PCB"
