File: pcb/hypnos/hypnos.sch (KiCad schematic (older format))
At the start: 9 parts, among them J1 Shutdown_Switch, J2 User_Input, J3 Debug_Conn, Q1 FDN361BN, SW1 Reset_Switch, U1 RV-3028-C7, U2 BT840F

Commit message: backup work
Parts:
- removed BT1: BK-883, Hypnos:BAT_BK-883, symbol Hypnos:BK-883
- removed J1: Shutdown_Switch, Connector_PinHeader_2.54mm:PinHeader_1x02_P2.54mm_Horizontal, symbol Connector:Conn_01x02_Male
- removed J2: User_Input, Connector_PinHeader_2.54mm:PinHeader_1x02_P2.54mm_Horizontal, symbol Connector:Conn_01x02_Male
- added BT1: BC-2003-TR, Hypnos:BC-2003-TR, symbol Hypnos:BC-2003-TR
- added J1: Motherboard_IO, Hypnos:Conn-Female-RightAnglex3-SMD, symbol Connector:Conn_01x03_Male
- J3: footprint Connector_PinHeader_2.54mm:PinHeader_1x07_P2.54mm_Horizontal -> Hypnos:Conn-Female-RightAnglex7-SMD
- Q1: value FDN361BN -> NDS351NCT; footprint Hypnos:FDN361BN -> Package_TO_SOT_SMD:SOT-323_SC-70_Handsoldering; symbol Hypnos:FDN361BN -> Hypnos:NDS351NCT
Connections:
- net GND: now also Q1.2 (S), BT1.2 (-), J1.3 (Pin_3)
- net VDD: now also BT1.1 (+), BT1.3 (+)
- net at U2.11 (P0.11): now also SW1.1
- net at U2.13 (P0.13): no longer SW1.1
- net at U2.5 (P0.02/AIN0): now also U1.2 (~INT); no longer Q1.1 (G)
- net USER_INPUT: now reaches U2.6 (P0.03/AIN1)
- net USER_INPUT: now also J1.1 (Pin_1)
- net OFF_SWITCH_CTRL: now reaches U2.7 (P0.09)
- net OFF_SWITCH_CTRL: now also Q1.1 (G); no longer U1.2 (~INT)
- net OFF_SWITCH: now reaches Q1.3 (D)
- net OFF_SWITCH: now also J1.2 (Pin_2)
Other:
- moved on the sheet: SW1
Changed lines of the file:
@@
 L Switch:SW_Push SW1
 U 1 1 5ED86397
-P 9700 2700
-F 0 "SW1" H 9700 2650 50  0000 C CNN
-F 1 "Reset_Switch" H 9700 2550 50  0000 C CNN
-F 2 "Hypnos:SW_KSR223GLFG" H 9700 2900 50  0001 C CNN
-F 3 "~" H 9700 2900 50  0001 C CNN
-	1    9700 2700
-	1    0    0    -1
-$EndComp
-$Comp
-L Connector:Conn_01x02_Male J2
-U 1 1 5ED8DE76
-P 2850 3050
-F 0 "J2" H 2958 3231 50  0000 C CNN
-F 1 "User_Input" H 2958 3140 50  0000 C CNN
-F 2 "Connector_PinHeader_2.54mm:PinHeader_1x02_P2.54mm_Horizontal" H 2850 3050 50  0001 C CNN
-F 3 "~" H 2850 3050 50  0001 C CNN
-	1    2850 3050
+P 9700 3000
+F 0 "SW1" H 9700 2950 50  0000 C CNN
+F 1 "Reset_Switch" H 9700 2850 50  0000 C CNN
+F 2 "Hypnos:SW_KSR223GLFG" H 9700 3200 50  0001 C CNN
+F 3 "~" H 9700 3200 50  0001 C CNN
+	1    9700 3000
 	1    0    0    -1
 $EndComp
@@
 $EndComp
 $Comp
-L Connector:Conn_01x02_Male J1
-U 1 1 5ED8D7F7
-P 2500 1950
-F 0 "J1" H 2608 2131 50  0000 C CNN
-F 1 "Shutdown_Switch" H 2608 2040 50  0000 C CNN
-F 2 "Connector_PinHeader_2.54mm:PinHeader_1x02_P2.54mm_Horizontal" H 2500 1950 50  0001 C CNN
-F 3 "~" H 2500 1950 50  0001 C CNN
-	1    2500 1950
-	1    0    0    -1
-$EndComp
-$Comp
 L power:GND #PWR03
 U 1 1 5EE28315
-P 1750 1500
-F 0 "#PWR03" H 1750 1250 50  0001 C CNN
-F 1 "GND" H 1755 1327 50  0000 C CNN
-F 2 "" H 1750 1500 50  0001 C CNN
-F 3 "" H 1750 1500 50  0001 C CNN
-	1    1750 1500
+P 1850 1500
+F 0 "#PWR03" H 1850 1250 50  0001 C CNN
+F 1 "GND" H 1855 1327 50  0000 C CNN
+F 2 "" H 1850 1500 50  0001 C CNN
+F 3 "" H 1850 1500 50  0001 C CNN
+	1    1850 1500
 	0    -1   -1   0
 $EndComp
@@
 NoConn ~ 2300 2500
 $Comp
-L Hypnos:FDN361BN Q1
+L Hypnos:NDS351NCT Q1
 U 1 1 5ED7D825
 P 3250 1950
 F 0 "Q1" H 3348 1996 50  0000 L CNN
-F 1 "FDN361BN" H 3348 1905 50  0000 L CNN
-F 2 "Hypnos:FDN361BN" H 3250 1950 50  0001 L BNN
+F 1 "NDS351NCT" H 3348 1905 50  0000 L CNN
+F 2 "Package_TO_SOT_SMD:SOT-323_SC-70_Handsoldering" H 3250 1950 50  0001 L BNN
 F 3 "" H 3250 1950 50  0001 C CNN
 	1    3250 1950
 	1    0    0    -1
 $EndComp
-$Comp
-L power:GND #PWR07
-U 1 1 5EE59FFE
-P 3050 3150
-F 0 "#PWR07" H 3050 2900 50  0001 C CNN
-F 1 "GND" V 3055 3022 50  0000 R CNN
-F 2 "" H 3050 3150 50  0001 C CNN
-F 3 "" H 3050 3150 50  0001 C CNN
-	1    3050 3150
-	0    -1   -1   0
-$EndComp
-Wire Wire Line
-	4150 2900 3450 2900
-Wire Wire Line
-	3450 2900 3450 3050
-Wire Wire Line
-	3450 3050 3050 3050
-Wire Wire Line
-	2700 2050 2800 2050
-Wire Wire Line
-	2800 2050 2800 2250
-Wire Wire Line
-	2800 2250 3250 2250
-Wire Wire Line
-	3250 2250 3250 2150
-Wire Wire Line
-	2700 1950 2950 1950
-Wire Wire Line
-	2950 1950 2950 1750
-Wire Wire Line
-	2950 1750 3250 1750
-Wire Wire Line
-	3050 1650 3050 2050
-Wire Wire Line
-	4150 2800 3950 2800
-Wire Wire Line
-	3950 2800 3950 1650
-Wire Wire Line
-	3050 1650 3950 1650
 Wire Wire Line
 	3700 2400 4150 2400
 Wire Wire Line
 	3700 2500 4150 2500
-Wire Wire Line
-	3700 2600 3850 2600
-Wire Wire Line
-	3850 2600 3850 3000
-Wire Wire Line
-	3850 3000 4150 3000
 $Comp
 L power:GND #PWR08
@@
 	3750 2700 3700 2700
 Wire Wire Line
-	9500 2700 9150 2700
+	9500 3000 9150 3000
 $Comp
 L power:GND #PWR011
 U 1 1 5EE682B6
-P 9900 2700
-F 0 "#PWR011" H 9900 2450 50  0001 C CNN
-F 1 "GND" V 9905 2572 50  0000 R CNN
-F 2 "" H 9900 2700 50  0001 C CNN
-F 3 "" H 9900 2700 50  0001 C CNN
-	1    9900 2700
+P 9900 3000
+F 0 "#PWR011" H 9900 2750 50  0001 C CNN
+F 1 "GND" V 9905 2872 50  0000 R CNN
+F 2 "" H 9900 3000 50  0001 C CNN
+F 3 "" H 9900 3000 50  0001 C CNN
+	1    9900 3000
 	0    -1   -1   0
 $EndComp
@@
 	1850 2600 1950 2600
 NoConn ~ 9150 2900
-NoConn ~ 9150 3000
 $Comp
 L Connector:Conn_01x07_Male J3
@@
 F 0 "J3" H 10458 3181 50  0000 C CNN
 F 1 "Debug_Conn" H 10458 3090 50  0000 C CNN
-F 2 "Connector_PinHeader_2.54mm:PinHeader_1x07_P2.54mm_Horizontal" H 10350 2700 50  0001 C CNN
+F 2 "Hypnos:Conn-Female-RightAnglex7-SMD" H 10350 2700 50  0001 C CNN
 F 3 "~" H 10350 2700 50  0001 C CNN
 	1    10350 2700
@@
 Wire Wire Line
 	10550 2900 11300 2900
-$Comp
-L Hypnos:BK-883 BT1
-U 1 1 5EF05217
-P 1450 1500
-F 0 "BT1" H 1475 1767 50  0000 C CNN
-F 1 "BK-883" H 1475 1676 50  0000 C CNN
-F 2 "Hypnos:BAT_BK-883" H 1600 1600 50  0001 L BNN
-F 3 "" H 1650 1400 50  0001 L BNN
-F 4 "" H 1500 1650 50  0001 L BNN "Field4"
-F 5 "" H 1600 1700 50  0001 L BNN "Field5"
-F 6 "" H 1650 1300 50  0001 L BNN "Field6"
-	1    1450 1500
-	1    0    0    -1
-$EndComp
 Wire Wire Line
 	1050 1550 1050 1500
@@
 	1150 1600 1200 1600
 $Comp
+L Hypnos:BC-2003-TR BT1
+U 1 1 5ED85647
+P 1400 1350
+F 0 "BT1" H 1475 1467 50  0000 C CNN
+F 1 "BC-2003-TR" H 1475 1376 50  0000 C CNN
+F 2 "Hypnos:BC-2003-TR" H 1400 1350 50  0001 C CNN
+F 3 "" H 1400 1350 50  0001 C CNN
+	1    1400 1350
+	1    0    0    -1
+$EndComp
+Wire Wire Line
+	1750 1500 1800 1500
+$Comp
 L power:PWR_FLAG #FLG03
 U 1 1 5EF1408F
-P 1700 1500
-F 0 "#FLG03" H 1700 1575 50  0001 C CNN
-F 1 "PWR_FLAG" H 1700 1673 50  0000 C CNN
-F 2 "" H 1700 1500 50  0001 C CNN
-F 3 "~" H 1700 1500 50  0001 C CNN
-	1    1700 1500
+P 1800 1500
+F 0 "#FLG03" H 1800 1575 50  0001 C CNN
+F 1 "PWR_FLAG" H 1800 1673 50  0000 C CNN
+F 2 "" H 1800 1500 50  0001 C CNN
+F 3 "~" H 1800 1500 50  0001 C CNN
+	1    1800 1500
 	-1   0    0    1
 $EndComp
+Connection ~ 1800 1500
+Wire Wire Line
+	1800 1500 1850 1500
+$Comp
+L Connector:Conn_01x03_Male J1
+U 1 1 5EDAA176
+P 3100 3550
+F 0 "J1" H 3208 3831 50  0000 C CNN
+F 1 "Motherboard_IO" H 3208 3740 50  0000 C CNN
+F 2 "Hypnos:Conn-Female-RightAnglex3-SMD" H 3100 3550 50  0001 C CNN
+F 3 "~" H 3100 3550 50  0001 C CNN
+	1    3100 3550
+	1    0    0    -1
+$EndComp
+$Comp
+L power:GND #PWR07
+U 1 1 5EDB98F3
+P 3300 3650
+F 0 "#PWR07" H 3300 3400 50  0001 C CNN
+F 1 "GND" H 3305 3477 50  0000 C CNN
+F 2 "" H 3300 3650 50  0001 C CNN
+F 3 "" H 3300 3650 50  0001 C CNN
+	1    3300 3650
+	0    -1   -1   0
+$EndComp
+Text Label 3650 2900 0    50   ~ 0
+USER_INPUT
+Text Label 3450 3450 0    50   ~ 0
+USER_INPUT
+Wire Wire Line
+	3300 3450 3450 3450
+$Comp
+L power:GND #PWR014
+U 1 1 5EDD0A45
+P 3250 2150
+F 0 "#PWR014" H 3250 1900 50  0001 C CNN
+F 1 "GND" H 3255 1977 50  0000 C CNN
+F 2 "" H 3250 2150 50  0001 C CNN
+F 3 "" H 3250 2150 50  0001 C CNN
+	1    3250 2150
+	1    0    0    -1
+$EndComp
+Text Label 3450 3550 0    50   ~ 0
+OFF_SWITCH
+Wire Wire Line
+	3300 3550 3450 3550
+Text Label 3250 1750 0    50   ~ 0
+OFF_SWITCH
+Wire Wire Line
+	3650 2900 4150 2900
+NoConn ~ 9150 2700
+Wire Wire Line
+	3700 2600 3900 2600
+Wire Wire Line
+	3900 2600 3900 2800
+Wire Wire Line
+	3900 2800 4150 2800
+Text Label 2350 2050 0    50   ~ 0
+OFF_SWITCH_CTRL
+Wire Wire Line
+	2350 2050 3050 2050
+Text Label 3000 3000 0    50   ~ 0
+OFF_SWITCH_CTRL
+Wire Wire Line
+	3000 3000 4150 3000
 $EndSCHEMATC
